File: jetson_gpio/Untitled/Untitled.kicad_pcb (KiCad board)
At the start: 2 copper layers, 34.3 x 71.1 mm, 36 parts, among them J1 Conn_01x10_Pin, J2 Conn_01x10_Pin, Q1 BC547B, Q2 BC547B, Q3 BC547B, Q4 BC547B, Q5 BC547B, Q6 BC547B, Q7 BC547B, Q8 BC547B

Commit message: update
Parts:
- moved Q5 3.87 mm to (81.3, 71.1), turned to -90 degrees
- moved Q6 3.87 mm to (81.3, 62.2), turned to -90 degrees
- moved Q7 3.87 mm to (81.3, 53.3), turned to -90 degrees
- moved Q8 3.87 mm to (81.3, 44.4), turned to -90 degrees
- moved Q1 3.87 mm to (81.3, 106.6), turned to -90 degrees
- moved Q2 3.87 mm to (81.3, 97.7), turned to -90 degrees
- moved Q3 3.87 mm to (81.3, 88.8), turned to -90 degrees
- moved Q4 3.87 mm to (81.3, 80.0), turned to -90 degrees
Routing:
- net GND: track 0.00 -> 3.59 mm
- net /VMA436_IN_8: track 22.1 -> 20.8 mm
- net /VMA436_IN_7: track 15.8 -> 14.4 mm
- net /VMA436_IN_3: track 17.2 -> 18.3 mm
- net /VMA436_IN_2: track 23.5 -> 24.7 mm
- net /VMA436_IN_1: track 29.9 -> 31.0 mm
- net /5V: track 128.1 -> 127.3 mm
- net /VMA436_IN_4: track 11.8 -> 12.3 mm
- net /VMA436_IN_6: track 11.3 -> 10.7 mm
- net /VMA436_IN_5: track 9.15 -> 9.70 mm
- net Net-(Q6-C): track 5.61 -> 5.10 mm
- net Net-(Q7-C): track 5.61 -> 5.10 mm
- net Net-(Q5-C): track 5.61 -> 5.10 mm
- net Net-(Q4-C): track 5.61 -> 5.10 mm
- net Net-(Q3-C): track 5.61 -> 5.10 mm
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Other:
- board size 34.3 x 71.1 mm -> 34.3 x 72.4 mm
